File: design/pdf_viewer/clock.kicad_sch (KiCad schematic)
At the start: 0 parts

Commit message: add footprint
Parts:
- added C6: 12pF, symbol Device:C_Small
- added C7, C8: C_Small, symbol Device:C_Small
- added R1: 1M, symbol Device:R_US
- added R2, R3: R_US, symbol Device:R_US
- added U3: CLOCK, Package_FBGA828, symbol rock:RK3399_clock
- added Y2: 24MHz, symbol Device:Crystal_GND24_Small
Connections:
- new net: C6.1, R1.1, U3.Y31 (XIN_OSC), Y2.1
- new net: C7.2, R2.1, Y2.3
- new net: C8.1, R3.2, U3.T30 (nPOR_u)
- new net: R1.2, R2.2, U3.Y30 (XOUT_OSC)
- new net BT_HOST_WAKE_L: U3.AA25 (SDIO0_INTn/GPIO0_A4_d)
- new net BT_REG_ON_H: U3.V30 (PMUIO2_VOLSEL/GPIO0_B1_d)
- new net GNDREF: C6.2, C7.1, C8.2, U3.P17 (PLL_AVSS), U3.Y29 (AVSS_48), Y2.2, Y2.4
- new net GPIO0_A2: U3.N24 (WIFI_26MHz/GPIO0_A2_d)
- new net GPIO0_B5/LED1_OUT: U3.P24 (TCPD_VBUS_SOURCE3/TCPD_VBUS_FDIS/GPIO0_B5_d)
- new net IR_RX: U3.P25 (PWM3A_IR/GPIO0_A6_d)
- new net MIPI_CSI1_PWN: U3.V26 (TCPD_VBUS_BDIS/GPIO0_B4_d)
- new net MIPI_CSI1_RST: U3.U28 (SDMMC0_WRPT/TEST_CLKOUT2/GPIO0_B0_u)
- new net PWR_KEY_L: U3.V27 (EMMC_PWRON/GPIO0_A5_u)
- new net RESET_L: R3.1
- new net RTC_CLKO_SOC: U3.U31 (TEST_CLKOUT0/CLK32K_IN/GPIO0_A0_u)
- new net SDMMC0_DET_L: U3.V28 (SDMMC0_DET/GPIO0_A7_u)
- new net SDMMC0_PWR_H: U3.R29 (DDRIO_PWROFF/TCPD_CCDB_EN/GPIO0_A1_u)
- new net WIFI_HOST_WAKE_L: U3.V31 (SDIO0_WRPT/GPIO0_A3_d)
- new net WIFI_REG_ON_H: U3.W31 (GPIO0_B2_d)
- no-connect marks 0 -> 1
