File: design/pdf_viewer/pdf_viewer.kicad_sch (KiCad schematic)
At the start: 0 parts

Commit message: add footprint
Other:
- added sheet dsi-edp-converter (dsi-edp-converter.kicad_sch)
Changed lines of the file:
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@@
 	(paper "A3")
+	(sheet
+		(at 123.19 684.53)
+		(size 121.92 26.67)
+		(fields_autoplaced yes)
+		(stroke
+			(width 0.1524)
+			(type solid)
+		)
+		(fill
+			(color 0 0 0 0.0000)
+		)
+		(property "Sheetname" "dsi-edp-converter"
+			(at 123.19 683.8184 0)
+			(effects
+				(font
+					(size 1.27 1.27)
+				)
+				(justify left bottom)
+			)
+		)
+		(property "Sheetfile" "dsi-edp-converter.kicad_sch"
+			(at 123.19 711.7846 0)
+			(effects
+				(font
+					(size 1.27 1.27)
+				)
+				(justify left top)
+			)
+		)
+		(instances
+			(project "pdf_viewer"
+				(path "/aeb14311-f547-46aa-9ccf-c37d4e677946"
+					(page "4")
+				)
+			)
+		)
+	)
 	(sheet
 		(at 252.73 883.92)
