File: design/pdf_viewer/pdf_viewer.kicad_pcb (KiCad board)
At the start: 2 copper layers, 4 parts

Commit message: fix build error
for buildroot

debug

ldflags

correspond to old version

fixed warnings

fix warnings

fix warnigs
Parts:
- renumbered RK3399 to REF**
Routing:
- net VCC_DDR: track 8.86 -> 1.71 mm
- net VCC.DDR: track 0.00 -> 7.15 mm
- net GND: track 59.5 -> 59.1 mm, vias 0 -> 14
